Commit message: finished week 4

File: urdf/bot_front_caster.urdf (robot description, URDF)
Before this commit: robot bot, 7 links, 6 joints
Links:
- link axle: geometry visual mesh filename=package://me169/me169git/meshes/body_front_caster.stl
- link leftwheel: geometry visual mesh filename=package://me169/me169git/meshes/wheel.stl
- link rightwheel: geometry visual mesh filename=package://me169/me169git/meshes/wheel.stl

File: urdf/bot_front_wheels.urdf (robot description, URDF)
Before this commit: robot bot, 7 links, 6 joints
Links:
- link axle: geometry visual mesh filename=package://me169/me169git/meshes/body_front_wheels.stl
- link leftwheel: geometry visual mesh filename=package://me169/me169git/meshes/wheel.stl
- link rightwheel: geometry visual mesh filename=package://me169/me169git/meshes/wheel.stl
